Commit message: update

File: youbot_description/robots/youbot.urdf.xacro (robot description, xacro)
@@ -22,4 +22,6 @@
   <!-- sensors -->
   <xacro:include filename="$(find youbot_description)/urdf/sensors/hokuyo_urg04_laser.urdf.xacro"/>
+  <!-- sensors -->
+  <xacro:include filename="$(find youbot_description)/urdf/sensors/lds_lfcd_sensor.urdf.xacro"/>
   <!-- Now we can start using the macros xacro:included above to define the actual youbot -->
   <!-- The first use of a macro.  This one was defined in base.urdf.xacro above.
@@ -41,7 +43,11 @@
     <origin xyz="0 0 0" rpy="0 0 0" />
   </xacro:youbot_gripper>
-  <!-- base laser front -->
-  <xacro:hokuyo_urg04_laser name="base_laser_front" parent="base" ros_topic="base_scan" update_rate="10" min_angle="-1.57" max_angle="1.57">
+  <!-- base hokuyo_urg04_laser front -->
+  <!-- <xacro:hokuyo_urg04_laser name="base_laser_front" parent="base" ros_topic="base_scan" update_rate="10" min_angle="-1.57" max_angle="1.57">
     <origin xyz="0.3 0 -0.03" rpy="0 0 0"/>
-  </xacro:hokuyo_urg04_laser>
+  </xacro:hokuyo_urg04_laser> -->
+  <!-- base lds_lfcd_sensor front -->
+  <xacro:lds_lfcd_sensor name="base_laser_front" parent="base" ros_topic="base_scan" update_rate="1800" min_angle="-1.57" max_angle="1.57">
+    <origin xyz="0.315 0 -0.03" rpy="0 0 0"/>
+  </xacro:lds_lfcd_sensor>
 </robot>

File: youbot_description/urdf/materials.urdf.xacro (robot description, xacro)
@@ -28,3 +28,6 @@
     <color rgba="0.82 0.82 0.82 1.0"/>
   </material>
+  <material name="dark">
+    <color rgba="0.3 0.3 0.3 1.0"/>
+  </material>
 </robot>
