Commit message: Update and modified

File: youbot_description/robots/youbot_arm_only.urdf.xacro (robot description, xacro)
@@ -25,4 +25,12 @@
        is the world frame). For more, see http://www.ros.org/wiki/xacro -->
   <!-- foot for arm-->
+  <!-- Fix the warn: The root link base_link has an inertia specified in the URDF, but KDL does not support a root link with an inertia.
+  As a workaround, you can add an extra dummy link to your URDF. So to fix it, the base_parent_link and joint are added.-->
+  <link name="base_parent_link"/>
+  <joint name="base_joint" type="fixed" >
+	<origin xyz="0 0 0" rpy="0 0 0" />
+	<parent link="base_parent_link" />
+	<child link="base_link" />
+  </joint> --add by hxq
   <link name="base_link">
     <inertial>

File: youbot_description/urdf/youbot_arm/arm.transmission.xacro (robot description, xacro)
@@ -4,15 +4,16 @@
        xmlns:interface="http://playerstage.sourceforge.net/gazebo/xmlschema/#interface"
        xmlns:xacro="http://ros.org/wiki/xacro">
+	<xacro:property name="hardware_interface" value="hardware_interface/EffortJointInterface" />
 	<!-- reduction ratio doesn't affect the model-->
 	<!-- reduction ratio must not to be 0-->
 	<xacro:macro name="youbot_arm_transmission" params="name">
-		<transmission name="${name}_trans_1">
+	  <transmission name="${name}_trans_1">
       <type>transmission_interface/SimpleTransmission</type>
 			<actuator name="${name}_motor_1">
-        <hardwareInterface>EffortJointInterface</hardwareInterface>
+        <hardwareInterface>${hardware_interface}</hardwareInterface>
         <mechanicalReduction>1</mechanicalReduction>
       </actuator>
 			<joint name="${name}_joint_1">
-        <hardwareInterface>EffortJointInterface</hardwareInterface>
+        <hardwareInterface>${hardware_interface}</hardwareInterface>
       </joint>
 		</transmission>
@@ -20,9 +21,9 @@
       <type>transmission_interface/SimpleTransmission</type>
 			<actuator name="${name}_motor_2">
-        <hardwareInterface>EffortJointInterface</hardwareInterface>
+        <hardwareInterface>${hardware_interface}</hardwareInterface>
         <mechanicalReduction>1</mechanicalReduction>
       </actuator>
 			<joint name="${name}_joint_2">
-        <hardwareInterface>EffortJointInterface</hardwareInterface>
+        <hardwareInterface>${hardware_interface}</hardwareInterface>
       </joint>
 		</transmission>
@@ -30,9 +31,9 @@
       <type>transmission_interface/SimpleTransmission</type>
 			<actuator name="${name}_motor_3">
-        <hardwareInterface>EffortJointInterface</hardwareInterface>
+        <hardwareInterface>${hardware_interface}</hardwareInterface>
         <mechanicalReduction>1</mechanicalReduction>
       </actuator>
 			<joint name="${name}_joint_3">
-        <hardwareInterface>EffortJointInterface</hardwareInterface>
+        <hardwareInterface>${hardware_interface}</hardwareInterface>
       </joint>
 		</transmission>
@@ -40,9 +41,9 @@
       <type>transmission_interface/SimpleTransmission</type>
 			<actuator name="${name}_motor_4">
-        <hardwareInterface>EffortJointInterface</hardwareInterface>
+        <hardwareInterface>${hardware_interface}</hardwareInterface>
         <mechanicalReduction>1</mechanicalReduction>
       </actuator>
 			<joint name="${name}_joint_4">
-        <hardwareInterface>EffortJointInterface</hardwareInterface>
+        <hardwareInterface>${hardware_interface}</hardwareInterface>
       </joint>
 		</transmission>
@@ -50,9 +51,9 @@
       <type>transmission_interface/SimpleTransmission</type>
 			<actuator name="${name}_motor_5">
-        <hardwareInterface>EffortJointInterface</hardwareInterface>
+        <hardwareInterface>${hardware_interface}</hardwareInterface>
         <mechanicalReduction>1</mechanicalReduction>
       </actuator>
 			<joint name="${name}_joint_5">
-        <hardwareInterface>EffortJointInterface</hardwareInterface>
+        <hardwareInterface>${hardware_interface}</hardwareInterface>
       </joint>
 		</transmission>

File: youbot_description/urdf/youbot_arm/arm.urdf.xacro (robot description, xacro)
@@ -188,6 +188,6 @@
 			<!--<calibration rising="${arm_5_ref}" falling="${arm_5_ref}"/>-->
 			<dynamics damping="1" friction="1" />
-			<limit effort="1" velocity="${M_PI / 2.0}" lower="0" upper="${joint_5_limit}" />
-                        <safety_controller k_position="20" k_velocity="100" soft_lower_limit="0" soft_upper_limit="${joint_5_limit_soft}" />
+			<limit effort="${1.0}" velocity="${M_PI / 2.0}" lower="0" upper="${joint_5_limit}" />
+            <safety_controller k_position="20" k_velocity="100" soft_lower_limit="0" soft_upper_limit="${joint_5_limit_soft}" />
 		</joint>
 		<link name="${name}_link_5">

File: youbot_description/urdf/youbot_base/base.transmission.xacro (robot description, xacro)
@@ -11,9 +11,9 @@
       <type>transmission_interface/SimpleTransmission</type>
 			<actuator name="wheel_motor_fl">
-        <hardwareInterface>VelocityJointInterface</hardwareInterface>
+        <hardwareInterface>hardware_interface/VelocityJointInterface</hardwareInterface>
         <mechanicalReduction>${wheel_mechanical_reduction}</mechanicalReduction>
       </actuator>
 			<joint name="wheel_joint_fl">
-        <hardwareInterface>VelocityJointInterface</hardwareInterface>
+        <hardwareInterface>hardware_interface/VelocityJointInterface</hardwareInterface>
       </joint>
 		</transmission>
@@ -21,9 +21,9 @@
       <type>transmission_interface/SimpleTransmission</type>
    	  <actuator name="caster_motor_fl">
-        <hardwareInterface>VelocityJointInterface</hardwareInterface>
+        <hardwareInterface>hardware_interface/VelocityJointInterface</hardwareInterface>
         <mechanicalReduction>${caster_mechanical_reduction}</mechanicalReduction>
       </actuator>
       <joint name="caster_joint_fl">
-        <hardwareInterface>VelocityJointInterface</hardwareInterface>
+        <hardwareInterface>hardware_interface/VelocityJointInterface</hardwareInterface>
       </joint>
     </transmission>
@@ -32,9 +32,9 @@
       <type>transmission_interface/SimpleTransmission</type>
 		  <actuator name="wheel_motor_fr">
-        <hardwareInterface>VelocityJointInterface</hardwareInterface>
+        <hardwareInterface>hardware_interface/VelocityJointInterface</hardwareInterface>
         <mechanicalReduction>${wheel_mechanical_reduction}</mechanicalReduction>
       </actuator>
 		  <joint name="wheel_joint_fr">
-        <hardwareInterface>VelocityJointInterface</hardwareInterface>
+        <hardwareInterface>hardware_interface/VelocityJointInterface</hardwareInterface>
       </joint>
 	  </transmission>
@@ -42,9 +42,9 @@
       <type>transmission_interface/SimpleTransmission</type>
       <actuator name="caster_motor_fr" >
-        <hardwareInterface>VelocityJointInterface</hardwareInterface>
+        <hardwareInterface>hardware_interface/VelocityJointInterface</hardwareInterface>
         <mechanicalReduction>${caster_mechanical_reduction}</mechanicalReduction>
       </actuator>
       <joint name="caster_joint_fr">
-        <hardwareInterface>VelocityJointInterface</hardwareInterface>
+        <hardwareInterface>hardware_interface/VelocityJointInterface</hardwareInterface>
       </joint>
     </transmission>
@@ -53,9 +53,9 @@
       <type>transmission_interface/SimpleTransmission</type>
 	    <actuator name="wheel_motor_bl" >
-        <hardwareInterface>VelocityJointInterface</hardwareInterface>
+        <hardwareInterface>hardware_interface/VelocityJointInterface</hardwareInterface>
         <mechanicalReduction>${wheel_mechanical_reduction}</mechanicalReduction>
       </actuator>
 	    <joint name="wheel_joint_bl">
-        <hardwareInterface>VelocityJointInterface</hardwareInterface>
+        <hardwareInterface>hardware_interface/VelocityJointInterface</hardwareInterface>
       </joint>
 	  </transmission>
@@ -63,9 +63,9 @@
       <type>transmission_interface/SimpleTransmission</type>
       <actuator name="caster_motor_bl" >
-        <hardwareInterface>VelocityJointInterface</hardwareInterface>
+        <hardwareInterface>hardware_interface/VelocityJointInterface</hardwareInterface>
         <mechanicalReduction>${caster_mechanical_reduction}</mechanicalReduction>
       </actuator>
       <joint name="caster_joint_bl">
-        <hardwareInterface>VelocityJointInterface</hardwareInterface>
+        <hardwareInterface>hardware_interface/VelocityJointInterface</hardwareInterface>
       </joint>
     </transmission>
@@ -74,9 +74,9 @@
       <type>transmission_interface/SimpleTransmission</type>
 	    <actuator name="wheel_motor_br" >
-        <hardwareInterface>VelocityJointInterface</hardwareInterface>
+        <hardwareInterface>hardware_interface/VelocityJointInterface</hardwareInterface>
         <mechanicalReduction>${wheel_mechanical_reduction}</mechanicalReduction>
       </actuator>
 		  <joint name="wheel_joint_br">
-        <hardwareInterface>VelocityJointInterface</hardwareInterface>
+        <hardwareInterface>hardware_interface/VelocityJointInterface</hardwareInterface>
       </joint>
 	  </transmission>
@@ -84,9 +84,9 @@
       <type>transmission_interface/SimpleTransmission</type>
       <actuator name="caster_motor_br" >
-        <hardwareInterface>VelocityJointInterface</hardwareInterface>
+        <hardwareInterface>hardware_interface/VelocityJointInterface</hardwareInterface>
         <mechanicalReduction>${caster_mechanical_reduction}</mechanicalReduction>
       </actuator>
       <joint name="caster_joint_br">
-        <hardwareInterface>VelocityJointInterface</hardwareInterface>
+        <hardwareInterface>hardware_interface/VelocityJointInterface</hardwareInterface>
       </joint>
     </transmission>

File: youbot_description/urdf/youbot_base/base.urdf.xacro (robot description, xacro)
@@ -6,5 +6,5 @@
   <!-- sensors -->
   <xacro:include filename="$(find youbot_description)/urdf/youbot_base/base.gazebo.xacro"/>
-  <xacro:include filename="$(find youbot_description)/urdf/youbot_base/base.transmission.xacro"/>
+  <!-- <xacro:include filename="$(find youbot_description)/urdf/youbot_base/base.transmission.xacro"/> --> because the base dosen't use ros_control
   <!-- simplified box collision geometry for base -->
   <xacro:property name="base_size_x" value="0.570"/>
@@ -274,5 +274,5 @@
     <!-- extensions -->
     <xacro:youbot_base_gazebo/>
-    <xacro:youbot_base_transmission/>
+    <!-- <xacro:youbot_base_transmission/> -->
   </xacro:macro>
 </robot>

File: youbot_description/urdf/youbot_gripper/gripper.transmission.xacro (robot description, xacro)
@@ -8,9 +8,9 @@
       <type>transmission_interface/SimpleTransmission</type>
 			<actuator name="${name}_finger_l_motor">
-        <hardwareInterface>EffortJointInterface</hardwareInterface>
+        <hardwareInterface>hardware_interface/EffortJointInterface</hardwareInterface>
         <mechanicalReduction>1</mechanicalReduction>
       </actuator>
 			<joint name="${name}_finger_joint_l">
-        <hardwareInterface>EffortJointInterface</hardwareInterface>
+        <hardwareInterface>hardware_interface/EffortJointInterface</hardwareInterface>
       </joint>
 		</transmission>
@@ -18,9 +18,9 @@
       <type>transmission_interface/SimpleTransmission</type>
 			<actuator name="${name}_finger_r_motor">
-        <hardwareInterface>EffortJointInterface</hardwareInterface>
+        <hardwareInterface>hardware_interface/EffortJointInterface</hardwareInterface>
         <mechanicalReduction>1</mechanicalReduction>
       </actuator>
 			<joint name="${name}_finger_joint_r">
-        <hardwareInterface>EffortJointInterface</hardwareInterface>
+        <hardwareInterface>hardware_interface/EffortJointInterface</hardwareInterface>
       </joint>
 		</transmission>

Commit message: Update

File: youbot_description/robots/youbot_arm_only.urdf.xacro (robot description, xacro)
@@ -16,4 +16,6 @@
   <!-- controller manager -->
   <xacro:include filename="$(find youbot_description)/controller/ros_controller.urdf.xacro" />
+  <!-- sensors -->
+  <xacro:include filename="$(find youbot_description)/urdf/sensors/xtion_pro_live.urdf.xacro"/>  add for grasping test
   <!-- Now we can start using the macros included above to define the actual youbot -->
   <!-- The first use of a macro.  This one was defined in base.urdf.xacro above.
@@ -46,3 +48,8 @@
     <origin xyz="0 0 0" rpy="0 0 0" />
   </xacro:youbot_gripper>
+  <!-- Define RGB-D sensor -->
+  <!-- <xacro:xtion_pro_live name="rgbd_camera" parent="base">
+    <origin xyz="0.5 0 2.5" rpy="0 ${75.0 * deg_to_rad} 0"/>
+    <origin xyz="0 0 0" rpy="${-90.0 * deg_to_rad} 0 ${-90.0 * deg_to_rad}"/>
+  </xacro:xtion_pro_live> -->  add for grasping test
 </robot>

File: youbot_description/urdf/common.xacro (robot description, xacro)
@@ -2,4 +2,5 @@
 <robot xmlns:xacro="http://ros.org/wiki/xacro">
 	<xacro:property name="M_PI" value="3.1415926535897931" />
+	<xacro:property name="deg_to_rad" value="0.01745329251994329577"/>  add by hxq
 	<!-- Casters -->
 	<xacro:property name="cal_caster_fl" value="0.0" />

File: youbot_description/urdf/youbot_arm/arm.transmission.xacro (robot description, xacro)
@@ -4,4 +4,5 @@
        xmlns:interface="http://playerstage.sourceforge.net/gazebo/xmlschema/#interface"
        xmlns:xacro="http://ros.org/wiki/xacro">
+	<!-- EffortJointInterface, PositionJointInterface -->
 	<xacro:property name="hardware_interface" value="hardware_interface/EffortJointInterface" />
 	<!-- reduction ratio doesn't affect the model-->

File: youbot_description/urdf/youbot_arm/arm.urdf.xacro (robot description, xacro)
@@ -6,5 +6,5 @@
 	<xacro:include filename="$(find youbot_description)/urdf/youbot_arm/arm.gazebo.xacro" />
 	<xacro:include filename="$(find youbot_description)/urdf/youbot_arm/arm.transmission.xacro" />
-        <xacro:include filename="$(find youbot_description)/urdf/youbot_arm/limits.urdf.xacro" />
+    <xacro:include filename="$(find youbot_description)/urdf/youbot_arm/limits.urdf.xacro" />
 	<xacro:macro name="youbot_arm" params="parent name *origin">
 		<!-- joint between base_link and arm_0_link -->
@@ -50,5 +50,5 @@
 			<!--effort - N, N*m-->
 			<!--velocity - m/s, rad/s-->
-			<safety_controller k_position="20" k_velocity="${9.5/M_PI / 2.0}" soft_lower_limit="${threshold}" soft_upper_limit="${joint_1_limit_soft}" />
+			<!-- <safety_controller k_position="20" k_velocity="${9.5/M_PI / 2.0}" soft_lower_limit="${threshold}" soft_upper_limit="${joint_1_limit_soft}" /> -->
 			<!--k_position N/m, N/rad-->
 			<!--k_velocity N*s/m, N*s*m/rad-->
@@ -85,5 +85,5 @@
 			<dynamics damping="1" friction="1" />
 			<limit effort="${9.5}" velocity="${M_PI / 2.0}" lower="0" upper="${joint_2_limit}"/>
-                        <safety_controller k_position="20" k_velocity="${2*9.5/M_PI}" soft_lower_limit="${threshold}" soft_upper_limit="${joint_2_limit_soft}" />
+            <!-- <safety_controller k_position="20" k_velocity="${2*9.5/M_PI}" soft_lower_limit="${threshold}" soft_upper_limit="${joint_2_limit_soft}" /> -->
 		</joint>
 		<link name="${name}_link_2">
@@ -116,5 +116,5 @@
 			<dynamics damping="1" friction="1" />
 			<limit effort="${6}" velocity="${M_PI / 2.0}" lower="-${joint_3_limit}" upper="0"/>
-                        <safety_controller k_position="20" k_velocity="50" soft_lower_limit="-${joint_3_limit_soft}" soft_upper_limit="${threshold}" />
+            <safety_controller k_position="20" k_velocity="50" soft_lower_limit="-${joint_3_limit_soft}" soft_upper_limit="${threshold}" />
 		</joint>-->
 		<joint name="${name}_joint_3" type="revolute">
@@ -125,5 +125,5 @@
 			<dynamics damping="1" friction="1" />
 			<limit effort="${6}" velocity="${M_PI / 2.0}" lower="-${joint_3_limit}" upper="0"/>
-                        <safety_controller k_position="20" k_velocity="50" soft_lower_limit="-${joint_3_limit_soft}" soft_upper_limit="-${threshold}" />
+            <!-- <safety_controller k_position="20" k_velocity="50" soft_lower_limit="-${joint_3_limit_soft}" soft_upper_limit="-${threshold}" /> -->
 		</joint>
 		<link name="${name}_link_3">
@@ -155,7 +155,7 @@
 			<axis xyz="0 1 0" />
 			<!--<calibration rising="${arm_4_ref}" falling="${arm_4_ref}"/>-->
-			<dynamics damping="1" friction="1" />
+			<dynamics damping="1" friction="0.5" />
 			<limit effort="${2}" velocity="${M_PI / 2.0}" lower="0" upper="${joint_4_limit}"/>
-			<safety_controller k_position="20" k_velocity="100" soft_lower_limit="0" soft_upper_limit="${joint_4_limit_soft}" />
+			<!-- <safety_controller k_position="20" k_velocity="100" soft_lower_limit="0" soft_upper_limit="${joint_4_limit_soft}" /> -->
 		</joint>
 		<link name="${name}_link_4">
@@ -187,7 +187,7 @@
 			<axis xyz="0 0 -1" />
 			<!--<calibration rising="${arm_5_ref}" falling="${arm_5_ref}"/>-->
-			<dynamics damping="1" friction="1" />
+			<dynamics damping="1" friction="0.1" /> modify to 0.1, to avoid turning too slowly
 			<limit effort="${1.0}" velocity="${M_PI / 2.0}" lower="0" upper="${joint_5_limit}" />
-            <safety_controller k_position="20" k_velocity="100" soft_lower_limit="0" soft_upper_limit="${joint_5_limit_soft}" />
+            <!-- <safety_controller k_position="20" k_velocity="100" soft_lower_limit="0" soft_upper_limit="${joint_5_limit_soft}" /> -->
 		</joint>
 		<link name="${name}_link_5">

File: youbot_description/urdf/youbot_arm/limits.urdf.xacro (robot description, xacro)
@@ -16,10 +16,10 @@
 	<xacro:property name="joint_5_limit_soft" value="${M_PI * (167.5 + 167.5) / 180 - threshold}" />
 	<!-- dynamic properties : mass (kg) Alu data sheet -->
-	<xacro:property name="link_0_mass" value="0.845" />
+	<!-- <xacro:property name="link_0_mass" value="0.845" />
 	<xacro:property name="link_1_mass" value="2.412" />
 	<xacro:property name="link_2_mass" value="1.155" />
 	<xacro:property name="link_3_mass" value="0.934" />
 	<xacro:property name="link_4_mass" value="0.877" />
-	<xacro:property name="link_5_mass" value="0.251" />
+	<xacro:property name="link_5_mass" value="0.251" /> -->
 	<!--<xacro:property name="link_0_mass" value="0.845" />
 	<xacro:property name="link_1_mass" value="0.1" />
@@ -28,9 +28,16 @@
 	<xacro:property name="link_4_mass" value="0.1" />
 	<xacro:property name="link_5_mass" value="0.1" />-->
+	<!-- update by mas-group -->
+	<xacro:property name="link_0_mass" value="0.961" />
+	<xacro:property name="link_1_mass" value="1.390" />
+	<xacro:property name="link_2_mass" value="1.318" />
+	<xacro:property name="link_3_mass" value="0.821" />
+	<xacro:property name="link_4_mass" value="0.769" />
+	<xacro:property name="link_5_mass" value="0.687" />
 	<!-- TODO: add inertia tensor-->
 	<xacro:macro name="default_origin">
         	<origin xyz="0 0 0" rpy="0 0 0"/> <!-- no data known -->
 	</xacro:macro>
-	<xacro:macro name="link_default_inertia_tensor">
+	<!-- <xacro:macro name="link_default_inertia_tensor">
 		<origin xyz="0 0 0"
 			rpy="0 0 0" />
@@ -61,4 +68,35 @@
 			rpy="0 0 0" />
 		<inertia ixx="0.000280" ixy="0.000000" ixz="0.000000" iyy="0.000339" iyz="0.000000" izz="0.000119" />
+	</xacro:macro> -->
+	<!-- update by mas-group -->
+	<xacro:macro name="link_default_inertia_tensor">
+		<origin xyz="0 0 0"
+			rpy="0 0 0" />
+		<inertia ixx="1.0" ixy="0.0" ixz="0.0" iyy="1.0" iyz="0.0" izz="1.0"/>
+	</xacro:macro>
+	<xacro:macro name="link_1_inertia_tensor">
+		<origin xyz="${14.89/1000} ${2.13/1000} ${2.13/1000}"
+			rpy="0 0 0" />
+		<inertia ixx="0.0029525" ixy="0.0" ixz="0.0" iyy="0.0060091" iyz="0.0" izz="0.0058821"/>
+	</xacro:macro>
+	<xacro:macro name="link_2_inertia_tensor">
+		<origin xyz="${10.53/1000} ${-30.7/1000} ${85.97/1000}"
+			rpy="0 0 0" />
+		<inertia ixx="0.0031145" ixy="0.0" ixz="0.0" iyy="0.0005843" iyz="0.0" izz="0.0031631"/>
+	</xacro:macro>
+	<xacro:macro name="link_3_inertia_tensor">
+		<origin xyz="${0.1/1000} ${20.7/1000} ${71.07/1000}"
+			rpy="0 0 0" />
+		<inertia ixx="0.00172767" ixy="0.0" ixz="0.0" iyy="0.00041967" iyz="0.0" izz="0.0018468"/>
+	</xacro:macro>
+	<xacro:macro name="link_4_inertia_tensor">
+		<origin xyz="${0.11/1000} ${-20.0/1000} ${50.19/1000}"
+			rpy="0 0 0"  />
+		<inertia ixx="0.0006764" ixy="0.0" ixz="0.0" iyy="0.0010573" iyz="0.0" izz="0.0006610"/>
+	</xacro:macro>
+	<xacro:macro name="link_5_inertia_tensor">
+		<origin xyz="${0/1000} ${1.15/1000} ${-16.83/1000}"
+			rpy="0 0 0" />
+		<inertia ixx="0.0001934" ixy="0.0" ixz="0.0" iyy="0.0001602" iyz="0.0" izz="0.0000689"/>
 	</xacro:macro>
 </robot>
