Commit message: update youbot + 3d camera

File: youbot_description/robots/youbot_with_cam3d.urdf.xacro (robot description, xacro)
@@ -23,4 +23,7 @@
   <xacro:include filename="$(find youbot_description)/urdf/sensors/hokuyo_urg04_laser.urdf.xacro"/>
   <xacro:include filename="$(find youbot_description)/urdf/sensors/lds_lfcd_sensor.urdf.xacro"/>
+  <xacro:include filename="$(find youbot_description)/urdf/sensors/asus_xtion_camera.urdf.xacro"/>
+  <!-- sensor tower -->
+  <xacro:include filename="$(find youbot_description)/urdf/misc/camera_tower.urdf.xacro"/>
   <!-- Now we can start using the macros xacro:included above to define the actual youbot -->
   <!-- The first use of a macro.  This one was defined in base.urdf.xacro above.
@@ -30,5 +33,5 @@
        (e.g., base_link).  The xacro:included origin block is also an argument to the macro.  By convention,
        the origin block defines where the component is w.r.t its parent (in this case the parent
-       is the world frame). For more, see http://www.ros.org/wiki/xacro -->
+       is the w/home/hxq/Documents/Repository backup/mas-group/youbot_description/urdf/misc/camera_tower.urdf.xacroorld frame). For more, see http://www.ros.org/wiki/xacro -->
   <!-- foot for arm-->
   <xacro:youbot_base name="base"/>
@@ -50,3 +53,11 @@
     <origin xyz="0.315 0 -0.03" rpy="0 0 0"/>
   </xacro:lds_lfcd_sensor>
+  <!-- camera tower -->
+  <xacro:camera_tower name="camera_tower" parent="plate_link">
+    <origin xyz="-0.11 0.0 0.03" rpy="0 0 0" />
+  </xacro:camera_tower>
+  <!-- 3D camera on tower -->
+  <xacro:asus_xtion_camera name="tower_cam3d" parent="camera_tower_link" tilt="0.5">
+    <origin xyz="0 0 0.49" rpy="0 0 0" />
+  </xacro:asus_xtion_camera>
 </robot>

File: youbot_description/urdf/sensors/asus_xtion_camera.urdf.xacro (robot description, xacro)
@@ -1,5 +1,5 @@
 <?xml version="1.0"?>
 <root xmlns:xacro="http://playerstage.sourceforge.net/gazebo/xmlschema/#interface">
-  <xacro:include filename="$(find youbot_description)/urdf/sensors/asus_xtion_camera.gazebo.xacro" />
+  <xacro:include filename="$(find youbot_description)/urdf/sensors/asus_xtion_camera_new.gazebo.xacro" />
   <xacro:property name="eye_x_offset" value="0.03" />
   <xacro:property name="eye_y_offset" value="0.035" />

Commit message: Update

File: youbot_description/robots/youbot_with_cam3d.urdf.xacro (robot description, xacro)
@@ -58,5 +58,5 @@
   </xacro:camera_tower>
   <!-- 3D camera on tower -->
-  <xacro:asus_xtion_camera name="tower_cam3d" parent="camera_tower_link" tilt="0.5">
+  <xacro:asus_xtion_camera name="tower_cam3d" parent="camera_tower_link" tilt="0"> <!-- tower_cam3d, camera -->
     <origin xyz="0 0 0.49" rpy="0 0 0" />
   </xacro:asus_xtion_camera>

File: youbot_description/urdf/misc/camera_tower.urdf.xacro (robot description, xacro)
@@ -8,5 +8,5 @@
   <xacro:property name="camera_tower_depth" value="0.03" />
   <xacro:macro name="camera_tower" params="name parent *origin">
-  	<link name="${name}_link">
+    <link name="${name}_link">
       <inertial>
         <mass value="0.5" />

File: youbot_description/urdf/sensors/asus_xtion_camera.urdf.xacro (robot description, xacro)
@@ -19,5 +19,5 @@
   </xacro:macro>
   <xacro:macro name="asus_xtion_camera" params="name parent *origin tilt">
-  	<link name="${name}_foot_link">
+    <link name="${name}_foot_link">
       <inertial>
         <mass value="0.05" />
@@ -98,21 +98,21 @@
     </joint>
     <xacro:asus_xtion_eye suffix="depth" parent="${name}">
-		<origin xyz="${eye_x_offset} ${eye_y_offset - 0.02} 0" rpy="0 0 0" />
-	</xacro:asus_xtion_eye>
-	<xacro:asus_xtion_eye suffix="depth_optical" parent="${name}">
-		<origin xyz="${eye_x_offset} ${eye_y_offset - 0.02} 0" rpy="${-M_PI/2} 0 ${-M_PI/2}" />
-	</xacro:asus_xtion_eye>
-	<xacro:asus_xtion_eye suffix="rgb" parent="${name}">
-		<origin xyz="${eye_x_offset} ${eye_y_offset - 0.04} 0" rpy="0 0 0" />
-	</xacro:asus_xtion_eye>
-	<xacro:asus_xtion_eye suffix="rgb_optical" parent="${name}">
-		<origin xyz="${eye_x_offset} ${eye_y_offset - 0.04} 0" rpy="${-M_PI/2} 0 ${-M_PI/2}" />
-	</xacro:asus_xtion_eye>
-	<xacro:asus_xtion_eye suffix="laser" parent="${name}">
-		<origin xyz="${eye_x_offset} ${eye_y_offset - 0.09} 0" rpy="0 0 0" />
-	</xacro:asus_xtion_eye>
-	<xacro:asus_xtion_eye suffix="laser_optical" parent="${name}">
-		<origin xyz="${eye_x_offset} ${eye_y_offset - 0.09} 0" rpy="${M_PI/2} 0 ${-M_PI/2}" />
-	</xacro:asus_xtion_eye>
+       <origin xyz="${eye_x_offset} ${eye_y_offset - 0.02} 0" rpy="0 0 0" />
+    </xacro:asus_xtion_eye>
+    <xacro:asus_xtion_eye suffix="depth_optical" parent="${name}">
+      <origin xyz="${eye_x_offset} ${eye_y_offset - 0.02} 0" rpy="${-M_PI/2} 0 ${-M_PI/2}" />
+    </xacro:asus_xtion_eye>
+    <xacro:asus_xtion_eye suffix="rgb" parent="${name}">
+      <origin xyz="${eye_x_offset} ${eye_y_offset - 0.04} 0" rpy="0 0 0" />
+    </xacro:asus_xtion_eye>
+    <xacro:asus_xtion_eye suffix="rgb_optical" parent="${name}">
+      <origin xyz="${eye_x_offset} ${eye_y_offset - 0.04} 0" rpy="${-M_PI/2} 0 ${-M_PI/2}" />
+    </xacro:asus_xtion_eye>
+    <xacro:asus_xtion_eye suffix="laser" parent="${name}">
+      <origin xyz="${eye_x_offset} ${eye_y_offset - 0.09} 0" rpy="0 0 0" />
+    </xacro:asus_xtion_eye>
+    <xacro:asus_xtion_eye suffix="laser_optical" parent="${name}">
+      <origin xyz="${eye_x_offset} ${eye_y_offset - 0.09} 0" rpy="${M_PI/2} 0 ${-M_PI/2}" />
+    </xacro:asus_xtion_eye>
    <!-- for simulation -->
    <xacro:asus_xtion_camera_gazebo name="${name}" />
