Commit message: Update description and simulation

File: youbot_description/controller/ros_controller.urdf.xacro (robot description, xacro)
@@ -4,6 +4,6 @@
        xmlns:interface="http://playerstage.sourceforge.net/gazebo/xmlschema/#interface">
   <gazebo>
-	<plugin name="gazebo_ros_controller" filename="libgazebo_ros_control.so" >
-		<legacyModeNS>true</legacyModeNS>
+    <plugin name="gazebo_ros_controller" filename="libgazebo_ros_control.so" >
+        <legacyModeNS>true</legacyModeNS>
     </plugin>
   </gazebo>

File: youbot_description/robots/youbot.urdf.xacro (robot description, xacro)
@@ -3,5 +3,5 @@
        xmlns:controller="http://playerstage.sourceforge.net/gazebo/xmlschema/#controller"
        xmlns:interface="http://playerstage.sourceforge.net/gazebo/xmlschema/#interface"
-       xmlns:xacro="http://ros.org/wiki/xacro"
+       xmlns:xacro="http://www.ros.org/wiki/xacro/#interface"
        name="youbot" >
   <!-- The following xacro:included files set up definitions of parts of the robot body -->
@@ -47,6 +47,6 @@
   </xacro:hokuyo_urg04_laser> -->
   <!-- base lds_lfcd_sensor front -->
-  <xacro:lds_lfcd_sensor name="base_laser_front" parent="base" ros_topic="base_scan" update_rate="1800" min_angle="-1.57" max_angle="1.57">
+  <xacro:lds_lfcd_sensor name="base_laser_front" parent="base" ros_topic="base_scan" update_rate="10" min_angle="-1.57" max_angle="1.57">
     <origin xyz="0.315 0 -0.03" rpy="0 0 0"/>
-  </xacro:lds_lfcd_sensor>
+  </xacro:lds_lfcd_sensor> -->
 </robot>

File: youbot_description/robots/youbot_arm_only.urdf.xacro (robot description, xacro)
@@ -3,5 +3,5 @@
        xmlns:controller="http://playerstage.sourceforge.net/gazebo/xmlschema/#controller"
        xmlns:interface="http://playerstage.sourceforge.net/gazebo/xmlschema/#interface"
-       xmlns:xacro="http://ros.org/wiki/xacro"
+       xmlns:xacro="http://www.ros.org/wiki/xacro/#interface"
        name="youbot" >
   <!-- The following included files set up definitions of parts of the robot body -->

File: youbot_description/robots/youbot_base_only.urdf.xacro (robot description, xacro)
@@ -3,5 +3,5 @@
        xmlns:controller="http://playerstage.sourceforge.net/gazebo/xmlschema/#controller"
        xmlns:interface="http://playerstage.sourceforge.net/gazebo/xmlschema/#interface"
-       xmlns:xacro="http://ros.org/wiki/xacro"
+       xmlns:xacro="http://www.ros.org/wiki/xacro/#interface"
        name="youbot" >
   <!-- The following xacro:included files set up definitions of parts of the robot body -->

File: youbot_description/robots/youbot_dual_arm.urdf.xacro (robot description, xacro)
@@ -3,5 +3,5 @@
        xmlns:controller="http://playerstage.sourceforge.net/gazebo/xmlschema/#controller"
        xmlns:interface="http://playerstage.sourceforge.net/gazebo/xmlschema/#interface"
-       xmlns:xacro="http://ros.org/wiki/xacro"
+       xmlns:xacro="http://www.ros.org/wiki/xacro/#interface"
        name="youbot" >
   <!-- The following xacro:included files set up definitions of parts of the robot body -->
@@ -47,5 +47,5 @@
   </xacro:youbot_gripper>
   <!-- base laser front -->
-  <xacro:hokuyo_urg04_laser name="base_laser_front" parent="base" ros_topic="base_scan" update_rate="10" min_angle="-1.57" max_angle="1.57">
+  <xacro:hokuyo_urg04_laser name="base_laser_front" parent="base" ros_topic="scan_front" update_rate="10" min_angle="-1.57" max_angle="1.57">
     <origin xyz="0.3 0 -0.03" rpy="0 0 0"/>
   </xacro:hokuyo_urg04_laser>

File: youbot_description/robots/youbot_with_cam3d.urdf.xacro (robot description, xacro)
@@ -3,5 +3,5 @@
        xmlns:controller="http://playerstage.sourceforge.net/gazebo/xmlschema/#controller"
        xmlns:interface="http://playerstage.sourceforge.net/gazebo/xmlschema/#interface"
-       xmlns:xacro="http://ros.org/wiki/xacro"
+       xmlns:xacro="http://www.ros.org/wiki/xacro/#interface"
        name="youbot" >
   <!-- The following xacro:included files set up definitions of parts of the robot body -->
@@ -33,5 +33,5 @@
        (e.g., base_link).  The xacro:included origin block is also an argument to the macro.  By convention,
        the origin block defines where the component is w.r.t its parent (in this case the parent
-       is the w/home/hxq/Documents/Repository backup/mas-group/youbot_description/urdf/misc/camera_tower.urdf.xacroorld frame). For more, see http://www.ros.org/wiki/xacro -->
+       is the world frame). For more, see http://www.ros.org/wiki/xacro -->
   <!-- foot for arm-->
   <xacro:youbot_base name="base"/>
@@ -50,5 +50,5 @@
   </xacro:hokuyo_urg04_laser> -->
   <!-- base lds_lfcd_sensor front -->
-  <xacro:lds_lfcd_sensor name="base_laser_front" parent="base" ros_topic="base_scan" update_rate="1800" min_angle="-1.57" max_angle="1.57">
+  <xacro:lds_lfcd_sensor name="base_laser_front" parent="base" ros_topic="base_scan" update_rate="10" min_angle="-1.57" max_angle="1.57">
     <origin xyz="0.315 0 -0.03" rpy="0 0 0"/>
   </xacro:lds_lfcd_sensor>

File: youbot_description/urdf/common.xacro (robot description, xacro)
@@ -1,4 +1,4 @@
 <?xml version="1.0"?>
-<robot xmlns:xacro="http://ros.org/wiki/xacro">
+<robot xmlns:xacro="http://www.ros.org/wiki/xacro/#interface">
 	<xacro:property name="M_PI" value="3.1415926535897931" />
 	<xacro:property name="deg_to_rad" value="0.01745329251994329577"/>  add by hxq

File: youbot_description/urdf/materials.urdf.xacro (robot description, xacro)
@@ -1,32 +1,32 @@
 <?xml version="1.0"?>
 <robot>
-  <material name="Orange">
+  <material name="youBot/Orange">
     <color rgba="1.0 0.4 0.0 1.0"/>
   </material>
-  <material name="Grey">
+  <material name="youBot/Grey">
     <color rgba="0.7 0.7 0.7 1.0"/>
   </material>
-  <material name="DarkGrey">
+  <material name="youBot/DarkGrey">
     <color rgba="0.3 0.3 0.3 1.0"/>
   </material>
-  <material name="White">
+  <material name="youBot/White">
     <color rgba="1.0 1.0 1.0 1.0"/>
   </material>
-  <material name="Black">
+  <material name="youBot/Black">
     <color rgba="0.0 0.0 0.0 1.0"/>
   </material>
-  <material name="Red">
+  <material name="youBot/Red">
     <color rgba="1.0 0.0 0.0 1.0"/>
   </material>
-  <material name="Green">
+  <material name="youBot/Green">
     <color rgba="0.0 1.0 0.0 1.0"/>
   </material>
-  <material name="Blue">
+  <material name="youBot/Blue">
     <color rgba="0.0 0.0 0.8 1.0"/>
   </material>
-  <material name="LightGrey">
+  <material name="youBot/LightGrey">
     <color rgba="0.82 0.82 0.82 1.0"/>
   </material>
-  <material name="dark">
+  <material name="dark">  use for lds_lfcd
     <color rgba="0.3 0.3 0.3 1.0"/>
   </material>

File: youbot_description/urdf/misc/sensor_angle.urdf.xacro (robot description, xacro)
@@ -3,5 +3,5 @@
        xmlns:controller="http://playerstage.sourceforge.net/gazebo/xmlschema/#controller"
        xmlns:interface="http://playerstage.sourceforge.net/gazebo/xmlschema/#interface"
-       xmlns:xacro="http://ros.org/wiki/xacro">
+       xmlns:xacro="http://www.ros.org/wiki/xacro/#interface">
 	<xacro:property name="sensor_angle_width"  value="0.097" />
 	<xacro:property name="sensor_angle_height" value="0.0015" />

File: youbot_description/urdf/sensors/asus_xtion_camera.gazebo.xacro (robot description, xacro)
@@ -3,62 +3,85 @@
       xmlns:controller="http://playerstage.sourceforge.net/gazebo/xmlschema/#controller"
       xmlns:interface="http://playerstage.sourceforge.net/gazebo/xmlschema/#interface"
-      xmlns:xacro="http://ros.org/wiki/xacro">
+      xmlns:xacro="http://www.ros.org/wiki/xacro/#interface">
 <xacro:macro name="asus_xtion_camera_gazebo" params="name">
-  <xacro:asus_xtion_depth_camera_gazebo name="${name}" />
-  <xacro:asus_xtion_rgb_camera_gazebo name="${name}" />
-</xacro:macro>
-<xacro:macro name="asus_xtion_depth_camera_gazebo" params="name">
-  <gazebo reference="${name}_depth_frame">
-    <sensor:camera name="${name}_depth_frame_sensor">
-      <imageFormat>R8G8B8</imageFormat>
-      <imageSize>640 480</imageSize>
-      <hfov>57</hfov>
-      <nearClip>0.01</nearClip>
-      <farClip>5</farClip>
+  <gazebo reference="${name}_camera">
+  <sensor type="depth" name="${name}_depth_frame_sensor">
+    <always_on>true</always_on>
+    <update_rate>20.0</update_rate>
+    <camera>
+      <horizontal_fov>${57.0*M_PI/180.0}</horizontal_fov>
+      <image>
+        <format>R8G8B8</format>
+        <width>640</width>
+        <height>480</height>
+      </image>
+      <clip>
+        <near>0.1</near>
+        <far>5</far>
+      </clip>
+    </camera>
+    <plugin name="${name}_depth_frame_controller" filename="libgazebo_ros_openni_kinect.so">
+      <baseline>0.2</baseline>
+      <alwaysOn>true</alwaysOn>
       <updateRate>20.0</updateRate>
+      <cameraName>${name}_depth</cameraName>
+      <imageTopicName>/${name}/ir/image_raw</imageTopicName>
+      <cameraInfoTopicName>/${name}/ir/camera_info</cameraInfoTopicName>
+      <depthImageTopicName>/${name}/depth/image_raw</depthImageTopicName>
+      <depthImageCameraInfoTopicName>/${name}/depth/camera_info</depthImageCameraInfoTopicName>
+      <pointCloudTopicName>/${name}/depth/points</pointCloudTopicName>
+      <frameName>${name}_depth_optical_frame</frameName>
+      <pointCloudCutoff>0.5</pointCloudCutoff>
+      <distortionK1>0.00000001</distortionK1>
+      <distortionK2>0.00000001</distortionK2>
+      <distortionK3>0.00000001</distortionK3>
+      <distortionT1>0.00000001</distortionT1>
+      <distortionT2>0.00000001</distortionT2>
+      <CxPrime>0</CxPrime>
+      <Cx>0</Cx>
+      <Cy>0</Cy>
+      <focalLength>0</focalLength>
+      <hackBaseline>0</hackBaseline>
+    </plugin>
+  </sensor>
+  <sensor type="depth" name="${name}_rgb_frame_sensor">
+    <always_on>true</always_on>
+    <update_rate>20.0</update_rate>
+    <camera>
+      <horizontal_fov>${57.0*M_PI/180.0}</horizontal_fov>
+      <image>
+        <format>R8G8B8</format>
+        <width>640</width>
+        <height>480</height>
+      </image>
+      <clip>
+        <near>0.1</near>
+        <far>5</far>
+      </clip>
+    </camera>
+    <plugin name="${name}_rgb_frame_controller" filename="libgazebo_ros_openni_kinect.so">
       <baseline>0.2</baseline>
-      <controller:gazebo_ros_camera name="${name}_depth_frame_controller" plugin="libgazebo_ros_camera.so">
-        <alwaysOn>true</alwaysOn>
-        <updateRate>20.0</updateRate>
-        <imageTopicName>/camera/ir/image_raw</imageTopicName>
-        <cameraInfoTopicName>/camera/ir/camera_info</cameraInfoTopicName>
-        <depthImageTopicName>/camera/depth/image_raw</depthImageTopicName>
-        <depthImageInfoTopicName>/camera/depth/camera_info</depthImageInfoTopicName>
-        <pointCloudTopicName>/camera/depth/points</pointCloudTopicName>
-        <frameName>/${name}_depth_optical_frame</frameName>
-        <pointCloudCutoff>0.5</pointCloudCutoff>
-        <distortion_k1>0.00000001</distortion_k1>
-        <distortion_k2>0.00000001</distortion_k2>
-        <distortion_k3>0.00000001</distortion_k3>
-        <distortion_t1>0.00000001</distortion_t1>
-        <distortion_t2>0.00000001</distortion_t2>
-      </controller:gazebo_ros_camera>
-    </sensor:camera>
-  </gazebo>
-</xacro:macro>
-<xacro:macro name="asus_xtion_rgb_camera_gazebo" params="name">
-  <gazebo reference="${name}_rgb_frame">
-    <sensor:camera name="${name}_rgb_frame_sensor">
-      <imageFormat>R8G8B8</imageFormat>
-      <imageSize>640 480</imageSize>
-      <hfov>57</hfov>
-      <nearClip>0.01</nearClip>
-      <farClip>5</farClip>
+      <alwaysOn>true</alwaysOn>
       <updateRate>20.0</updateRate>
-      <baseline>0.2</baseline>
-      <controller:gazebo_ros_camera name="${name}_rgb_frame_controller" plugin="libgazebo_ros_camera.so">
-        <alwaysOn>true</alwaysOn>
-        <updateRate>20.0</updateRate>
-        <imageTopicName>/camera/rgb/image_raw</imageTopicName>
-        <cameraInfoTopicName>/camera/rgb/camera_info</cameraInfoTopicName>
-        <frameName>/${name}_rgb_optical_frame</frameName>
-        <pointCloudCutoff>0.5</pointCloudCutoff>
-        <distortion_k1>0.00000001</distortion_k1>
-        <distortion_k2>0.00000001</distortion_k2>
-        <distortion_k3>0.00000001</distortion_k3>
-        <distortion_t1>0.00000001</distortion_t1>
-        <distortion_t2>0.00000001</distortion_t2>
-      </controller:gazebo_ros_camera>
-    </sensor:camera>
+      <cameraName>${name}_rgb</cameraName>
+      <imageTopicName>/${name}/rgb/image_raw</imageTopicName>
+      <cameraInfoTopicName>/${name}/rgb/camera_info</cameraInfoTopicName>
+      <depthImageTopicName>/${name}/depth_registered/image_raw</depthImageTopicName>
+      <depthImageCameraInfoTopicName>/${name}/depth_registered/camera_info</depthImageCameraInfoTopicName>
+      <pointCloudTopicName>/${name}/depth_registered/points</pointCloudTopicName>
+      <frameName>${name}_rgb_optical_frame</frameName>
+      <pointCloudCutoff>0.5</pointCloudCutoff>
+      <distortionK1>0.00000001</distortionK1>
+      <distortionK2>0.00000001</distortionK2>
+      <distortionK3>0.00000001</distortionK3>
+      <distortionT1>0.00000001</distortionT1>
+      <distortionT2>0.00000001</distortionT2>
+      <CxPrime>0</CxPrime>
+      <Cx>0</Cx>
+      <Cy>0</Cy>
+      <focalLength>0</focalLength>
+      <hackBaseline>0</hackBaseline>
+    </plugin>
+  </sensor>
   </gazebo>
 </xacro:macro>

File: youbot_description/urdf/sensors/asus_xtion_camera.urdf.xacro (robot description, xacro)
@@ -1,5 +1,5 @@
 <?xml version="1.0"?>
 <root xmlns:xacro="http://playerstage.sourceforge.net/gazebo/xmlschema/#interface">
-  <xacro:include filename="$(find youbot_description)/urdf/sensors/asus_xtion_camera_new.gazebo.xacro" />
+  <xacro:include filename="$(find youbot_description)/urdf/sensors/asus_xtion_camera.gazebo.xacro" />
   <xacro:property name="eye_x_offset" value="0.03" />
   <xacro:property name="eye_y_offset" value="0.035" />

File: youbot_description/urdf/sensors/hokuyo_urg04_laser.gazebo.xacro (robot description, xacro)
@@ -3,5 +3,5 @@
        xmlns:controller="http://playerstage.sourceforge.net/gazebo/xmlschema/#controller"
        xmlns:interface="http://playerstage.sourceforge.net/gazebo/xmlschema/#interface"
-       xmlns:xacro="http://ros.org/wiki/xacro">
+       xmlns:xacro="http://www.ros.org/wiki/xacro/#interface">
   <xacro:macro name="hokuyo_urg04_laser_gazebo" params="name ros_topic update_rate min_angle max_angle">
     <gazebo reference="${name}_link">

File: youbot_description/urdf/sensors/hokuyo_urg04_laser.urdf.xacro (robot description, xacro)
@@ -3,5 +3,5 @@
        xmlns:controller="http://playerstage.sourceforge.net/gazebo/xmlschema/#controller"
        xmlns:interface="http://playerstage.sourceforge.net/gazebo/xmlschema/#interface"
-       xmlns:xacro="http://ros.org/wiki/xacro">
+       xmlns:xacro="http://www.ros.org/wiki/xacro/#interface">
   <xacro:include filename="$(find youbot_description)/urdf/sensors/hokuyo_urg04_laser.gazebo.xacro" />
   <xacro:macro name="hokuyo_urg04_laser" params="name parent *origin ros_topic update_rate min_angle max_angle">
@@ -19,16 +19,15 @@
       </inertial>
       <visual>
-      	<origin xyz="0 0 0" rpy="0 0 0" />
-	<geometry>
-		<mesh filename="package://youbot_description/meshes/sensors/hokuyo.dae" />
-	</geometry>
-	<material name="DarkGrey" />
+        <origin xyz="0 0 0" rpy="0 0 0" />
+        <geometry>
+          <mesh filename="package://youbot_description/meshes/sensors/hokuyo.dae" />
+        </geometry>
       </visual>
       <collision>
-		<origin xyz="0 0 0" rpy="0 0 0" />
-		<geometry>
-			<mesh filename="package://youbot_description/meshes/sensors/hokuyo_convex.dae" />
-		</geometry>
-	</collision>
+        <origin xyz="0 0 0" rpy="0 0 0" />
+        <geometry>
+          <mesh filename="package://youbot_description/meshes/sensors/hokuyo_convex.dae" />
+        </geometry>
+      </collision>
     </link>
     <!-- gazebo extensions -->

File: youbot_description/urdf/sensors/kinect_camera.gazebo.xacro (robot description, xacro)
@@ -3,5 +3,5 @@
       xmlns:controller="http://playerstage.sourceforge.net/gazebo/xmlschema/#controller"
       xmlns:interface="http://playerstage.sourceforge.net/gazebo/xmlschema/#interface"
-      xmlns:xacro="http://ros.org/wiki/xacro">
+      xmlns:xacro="http://www.ros.org/wiki/xacro/#interface">
 <xacro:macro name="kinect_camera_gazebo" params="name">
   <gazebo reference="${name}_camera">

File: youbot_description/urdf/sensors/kinect_camera.urdf.xacro (robot description, xacro)
@@ -3,5 +3,5 @@
       xmlns:controller="http://playerstage.sourceforge.net/gazebo/xmlschema/#controller"
       xmlns:interface="http://playerstage.sourceforge.net/gazebo/xmlschema/#interface"
-      xmlns:xacro="http://ros.org/wiki/xacro">
+      xmlns:xacro="http://www.ros.org/wiki/xacro/#interface">
   <xacro:include filename="$(find youbot_description)/urdf/sensors/kinect_camera.gazebo.xacro"/>
   <xacro:macro name="kinect_camera" params="name parent *origin">

File: youbot_description/urdf/sensors/microsoft_lifecam.gazebo.xacro (robot description, xacro)
@@ -3,5 +3,5 @@
       xmlns:controller="http://playerstage.sourceforge.net/gazebo/xmlschema/#controller"
       xmlns:interface="http://playerstage.sourceforge.net/gazebo/xmlschema/#interface"
-      xmlns:xacro="http://ros.org/wiki/xacro">
+      xmlns:xacro="http://www.ros.org/wiki/xacro/#interface">
 <xacro:macro name="microsoft_lifecam_gazebo" params="name">
   <gazebo reference="${name}_camera">

File: youbot_description/urdf/sensors/microsoft_lifecam.urdf.xacro (robot description, xacro)
@@ -3,5 +3,5 @@
       xmlns:controller="http://playerstage.sourceforge.net/gazebo/xmlschema/#controller"
       xmlns:interface="http://playerstage.sourceforge.net/gazebo/xmlschema/#interface"
-      xmlns:xacro="http://ros.org/wiki/xacro">
+      xmlns:xacro="http://www.ros.org/wiki/xacro/#interface">
   <xacro:include filename="$(find youbot_description)/urdf/sensors/microsoft_lifecam.gazebo.xacro"/>
   <xacro:macro name="microsoft_lifecam" params="name parent *origin">

File: youbot_description/urdf/youbot_arm/arm.gazebo.xacro (robot description, xacro)
@@ -3,28 +3,22 @@
        xmlns:controller="http://playerstage.sourceforge.net/gazebo/xmlschema/#controller"
        xmlns:interface="http://playerstage.sourceforge.net/gazebo/xmlschema/#interface"
-       xmlns:xacro="http://ros.org/wiki/xacro">
+       xmlns:xacro="http://www.ros.org/wiki/xacro/#interface">
 	<xacro:macro name="youbot_arm_gazebo" params="name">
 		<gazebo reference="${name}_link_0">
-			<material value="youbot/DarkGrey" />
 			<turnGravityOff>false</turnGravityOff>
 		</gazebo>
 		<gazebo reference="${name}_link_1">
-			<!--<material value="youbot/Orange" />-->
 			<turnGravityOff>false</turnGravityOff>
 		</gazebo>
 		<gazebo reference="${name}_link_2">
-			<!--<material value="youbot/Orange" />-->
 			<turnGravityOff>false</turnGravityOff>
 		</gazebo>
 		<gazebo reference="${name}_link_3">
-			<!--<material value="youbot/Orange" />-->
 			<turnGravityOff>false</turnGravityOff>
 		</gazebo>
 		<gazebo reference="${name}_link_4">
-			<!--<material value="youbot/Orange" />-->
 			<turnGravityOff>false</turnGravityOff>
 		</gazebo>
 		<gazebo reference="${name}_link_5">
-			<!--<material value="youbot/DarkGrey" />-->
 			<turnGravityOff>false</turnGravityOff>
 		</gazebo>

File: youbot_description/urdf/youbot_arm/arm.transmission.xacro (robot description, xacro)
@@ -3,60 +3,60 @@
        xmlns:controller="http://playerstage.sourceforge.net/gazebo/xmlschema/#controller"
        xmlns:interface="http://playerstage.sourceforge.net/gazebo/xmlschema/#interface"
-       xmlns:xacro="http://ros.org/wiki/xacro">
-	<!-- EffortJointInterface, PositionJointInterface -->
-	<xacro:property name="hardware_interface" value="hardware_interface/EffortJointInterface" />
+       xmlns:xacro="http://www.ros.org/wiki/xacro/#interface">
+  <!-- EffortJointInterface, PositionJointInterface -->
+  <xacro:property name="hardware_interface" value="hardware_interface/EffortJointInterface" />
 	<!-- reduction ratio doesn't affect the model-->
-	<!-- reduction ratio must not to be 0-->
-	<xacro:macro name="youbot_arm_transmission" params="name">
-	  <transmission name="${name}_trans_1">
+  <!-- reduction ratio must not to be 0-->
+  <xacro:macro name="youbot_arm_transmission" params="name">
+    <transmission name="${name}_trans_1">
       <type>transmission_interface/SimpleTransmission</type>
-			<actuator name="${name}_motor_1">
+      <actuator name="${name}_motor_1">
         <hardwareInterface>${hardware_interface}</hardwareInterface>
         <mechanicalReduction>1</mechanicalReduction>
       </actuator>
-			<joint name="${name}_joint_1">
+      <joint name="${name}_joint_1">
         <hardwareInterface>${hardware_interface}</hardwareInterface>
       </joint>
-		</transmission>
-		<transmission name="${name}_trans_2">
+    </transmission>
+    <transmission name="${name}_trans_2">
       <type>transmission_interface/SimpleTransmission</type>
-			<actuator name="${name}_motor_2">
+      <actuator name="${name}_motor_2">
         <hardwareInterface>${hardware_interface}</hardwareInterface>
         <mechanicalReduction>1</mechanicalReduction>
       </actuator>
-			<joint name="${name}_joint_2">
+      <joint name="${name}_joint_2">
         <hardwareInterface>${hardware_interface}</hardwareInterface>
       </joint>
-		</transmission>
-		<transmission name="${name}_trans_3">
+    </transmission>
+    <transmission name="${name}_trans_3">
       <type>transmission_interface/SimpleTransmission</type>
-			<actuator name="${name}_motor_3">
+      <actuator name="${name}_motor_3">
         <hardwareInterface>${hardware_interface}</hardwareInterface>
         <mechanicalReduction>1</mechanicalReduction>
       </actuator>
-			<joint name="${name}_joint_3">
+      <joint name="${name}_joint_3">
         <hardwareInterface>${hardware_interface}</hardwareInterface>
       </joint>
-		</transmission>
-		<transmission name="${name}_trans_4">
+    </transmission>
+    <transmission name="${name}_trans_4">
       <type>transmission_interface/SimpleTransmission</type>
-			<actuator name="${name}_motor_4">
+      <actuator name="${name}_motor_4">
         <hardwareInterface>${hardware_interface}</hardwareInterface>
         <mechanicalReduction>1</mechanicalReduction>
       </actuator>
-			<joint name="${name}_joint_4">
+      <joint name="${name}_joint_4">
         <hardwareInterface>${hardware_interface}</hardwareInterface>
       </joint>
-		</transmission>
-		<transmission name="${name}_trans_5">
+    </transmission>
+    <transmission name="${name}_trans_5">
       <type>transmission_interface/SimpleTransmission</type>
-			<actuator name="${name}_motor_5">
+      <actuator name="${name}_motor_5">
         <hardwareInterface>${hardware_interface}</hardwareInterface>
         <mechanicalReduction>1</mechanicalReduction>
       </actuator>
-			<joint name="${name}_joint_5">
+      <joint name="${name}_joint_5">
         <hardwareInterface>${hardware_interface}</hardwareInterface>
       </joint>
-		</transmission>
-	</xacro:macro>
+    </transmission>
+  </xacro:macro>
 </robot>
