Commit message: Update description and simulation

File: youbot_description/urdf/youbot_arm/arm.urdf.xacro (robot description, xacro)
@@ -3,8 +3,8 @@
         xmlns:controller="http://playerstage.sourceforge.net/gazebo/xmlschema/#controller"
         xmlns:interface="http://playerstage.sourceforge.net/gazebo/xmlschema/#interface"
-        xmlns:xacro="http://ros.org/wiki/xacro">
+        xmlns:xacro="http://www.ros.org/wiki/xacro/#interface">
 	<xacro:include filename="$(find youbot_description)/urdf/youbot_arm/arm.gazebo.xacro" />
 	<xacro:include filename="$(find youbot_description)/urdf/youbot_arm/arm.transmission.xacro" />
-    <xacro:include filename="$(find youbot_description)/urdf/youbot_arm/limits.urdf.xacro" />
+	<xacro:include filename="$(find youbot_description)/urdf/youbot_arm/limits.urdf.xacro" />
 	<xacro:macro name="youbot_arm" params="parent name *origin">
 		<!-- joint between base_link and arm_0_link -->
@@ -26,5 +26,5 @@
 					<mesh filename="package://youbot_description/meshes/youbot_arm/arm0.dae" />
 				</geometry>
-				<material name="DarkGrey" />
+				<material name="youBot/DarkGrey" />
 			</visual>
 			<collision>
@@ -50,5 +50,5 @@
 			<!--effort - N, N*m-->
 			<!--velocity - m/s, rad/s-->
-			<!-- <safety_controller k_position="20" k_velocity="${9.5/M_PI / 2.0}" soft_lower_limit="${threshold}" soft_upper_limit="${joint_1_limit_soft}" /> -->
+			<!--safety_controller k_position="20" k_velocity="${9.5/M_PI / 2.0}" soft_lower_limit="${threshold}" soft_upper_limit="${joint_1_limit_soft}" /-->
 			<!--k_position N/m, N/rad-->
 			<!--k_velocity N*s/m, N*s*m/rad-->
@@ -65,5 +65,5 @@
 					<mesh filename="package://youbot_description/meshes/youbot_arm/arm1.dae" />
 				</geometry>
-				<!--<material name="Orange" />-->
+				<material name="youBot/Orange" />
 			</visual>
 			<collision>
@@ -85,5 +85,5 @@
 			<dynamics damping="1" friction="1" />
 			<limit effort="${9.5}" velocity="${M_PI / 2.0}" lower="0" upper="${joint_2_limit}"/>
-            <!-- <safety_controller k_position="20" k_velocity="${2*9.5/M_PI}" soft_lower_limit="${threshold}" soft_upper_limit="${joint_2_limit_soft}" /> -->
+      <!--safety_controller k_position="20" k_velocity="${2*9.5/M_PI}" soft_lower_limit="${threshold}" soft_upper_limit="${joint_2_limit_soft}" /-->
 		</joint>
 		<link name="${name}_link_2">
@@ -97,5 +97,5 @@
 					<mesh filename="package://youbot_description/meshes/youbot_arm/arm2.dae" />
 				</geometry>
-				<material name="Orange" />
+				<material name="youBot/Orange" />
 			</visual>
 			<collision>
@@ -116,5 +116,5 @@
 			<dynamics damping="1" friction="1" />
 			<limit effort="${6}" velocity="${M_PI / 2.0}" lower="-${joint_3_limit}" upper="0"/>
-            <safety_controller k_position="20" k_velocity="50" soft_lower_limit="-${joint_3_limit_soft}" soft_upper_limit="${threshold}" />
+      <safety_controller k_position="20" k_velocity="50" soft_lower_limit="-${joint_3_limit_soft}" soft_upper_limit="${threshold}" />
 		</joint>-->
 		<joint name="${name}_joint_3" type="revolute">
@@ -124,6 +124,6 @@
 			<axis xyz="0 1 0"/>
 			<dynamics damping="1" friction="1" />
-			<limit effort="${6}" velocity="${M_PI / 2.0}" lower="-${joint_3_limit}" upper="0"/>
-            <!-- <safety_controller k_position="20" k_velocity="50" soft_lower_limit="-${joint_3_limit_soft}" soft_upper_limit="-${threshold}" /> -->
+			<limit effort="${6.0}" velocity="${M_PI / 2.0}" lower="-${joint_3_limit}" upper="0"/>
+      <!--safety_controller k_position="20" k_velocity="50" soft_lower_limit="-${joint_3_limit_soft}" soft_upper_limit="-${threshold}" /-->
 		</joint>
 		<link name="${name}_link_3">
@@ -137,5 +137,5 @@
 					<mesh filename="package://youbot_description/meshes/youbot_arm/arm3.dae" />
 				</geometry>
-				<material name="Orange" />
+				<material name="youBot/Orange" />
 			</visual>
 			<collision>
@@ -155,7 +155,7 @@
 			<axis xyz="0 1 0" />
 			<!--<calibration rising="${arm_4_ref}" falling="${arm_4_ref}"/>-->
-			<dynamics damping="1" friction="0.5" />
-			<limit effort="${2}" velocity="${M_PI / 2.0}" lower="0" upper="${joint_4_limit}"/>
-			<!-- <safety_controller k_position="20" k_velocity="100" soft_lower_limit="0" soft_upper_limit="${joint_4_limit_soft}" /> -->
+			<dynamics damping="1" friction="0.5" />  modified
+			<limit effort="${2.0}" velocity="${M_PI / 2.0}" lower="0" upper="${joint_4_limit}"/>
+			<!--safety_controller k_position="20" k_velocity="100" soft_lower_limit="0" soft_upper_limit="${joint_4_limit_soft}" /-->
 		</joint>
 		<link name="${name}_link_4">
@@ -169,5 +169,5 @@
 					<mesh filename="package://youbot_description/meshes/youbot_arm/arm4.dae" />
 				</geometry>
-				<material name="Orange" />
+				<material name="youBot/Orange" />
 			</visual>
 			<collision>
@@ -189,5 +189,5 @@
 			<dynamics damping="1" friction="0.1" /> modify to 0.1, to avoid turning too slowly
 			<limit effort="${1.0}" velocity="${M_PI / 2.0}" lower="0" upper="${joint_5_limit}" />
-            <!-- <safety_controller k_position="20" k_velocity="100" soft_lower_limit="0" soft_upper_limit="${joint_5_limit_soft}" /> -->
+      <!--safety_controller k_position="20" k_velocity="100" soft_lower_limit="0" soft_upper_limit="${joint_5_limit_soft}" /-->
 		</joint>
 		<link name="${name}_link_5">
@@ -201,5 +201,5 @@
 					<mesh filename="package://youbot_description/meshes/youbot_arm/arm5.dae" />
 				</geometry>
-				<material name="DarkGrey" />
+				<material name="youBot/DarkGrey" />
 			</visual>
 			<collision>
