Commit message: Update

File: youbot_description/urdf/youbot_base/base.urdf.xacro (robot description, xacro)
@@ -33,9 +33,11 @@
   <xacro:macro name="youbot_base" params="name">
     <link name="${name}_footprint">
-      <inertial>
+      <!-- Fix the warn: [ WARN] [1533277946.206920022, 0.246000000]: The root link base_footprint has an inertia specified in the URDF,
+      but KDL does not support a root link with an inertia.  As a workaround, you can add an extra dummy link to your URDF. -->
+      <!-- <inertial>
         <mass value="0.1"/>
         <origin xyz="0 0 ${-base_size_z / 2.0}" rpy="0 0 0"/>
         <inertia ixx="1.0" ixy="0.0" ixz="0.0" iyy="1.0" iyz="0.0" izz="1.0"/>
-      </inertial>
+      </inertial> -->
       <visual>
         <origin xyz="0 0 0" rpy="0 0 0"/>
